File: RCP Pi Hat.kicad_pcb (KiCad board)
At the start: 2 copper layers, 65 x 56 mm, 29 parts, among them J1 Debug Pins, U3 AMS1117-3.3

Commit message: V20240220
Routing:
- net +5V: track 29.9 -> 8.84 mm, vias 1 -> 6
- added copper zone on B.Cu, net +5V
Other:
- board text added: "V20240220"
- board text removed: "V20240216"
